File: Wii_RA.kicad_sch (KiCad schematic)
At the start: 4 parts, among them P1 GC_MEMCARD, U1 XIAO-ESP32-C3

Commit message: Add files via upload
Parts:
- BZ1: value SMT-0540-S-R -> 5x5 3v buzzer
- D1: DESCRIPTION ON SEMICONDUCTOR - - DIODE, SCHOTTKY, 1A, 40V, DO-214AC-2 -> (none)
- U1: value XIAO-ESP32-C3 -> XIAO-ESP32-S3
Changed lines of the file:
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@@
 			)
 		)
-		(property "Value" "SMT-0540-S-R"
+		(property "Value" "5x5 3v buzzer"
 			(at 98.806 123.444 90)
 			(show_name no)
@@
 			)
 		)
-		(property "Description" "DIODE SCHOTTKY 40V 1A SMA"
-			(at 101.6 91.44 0)
-			(hide yes)
-			(show_name no)
-			(do_not_autoplace no)
-			(effects
-				(font
-					(size 1.27 1.27)
-				)
+		(property "Description" "ON SEMICONDUCTOR - - DIODE, SCHOTTKY, 1A, 40V, DO-214AC-2"
+			(at 101.092 88.646 90)
+			(hide yes)
+			(show_name no)
+			(do_not_autoplace no)
+			(effects
+				(font
+					(size 1.27 1.27)
+				)
+				(justify right bottom)
 			)
 		)
@@
 		)
 		(property "MANUFACTURER PART NUMBER" "SS14"
-			(at 101.092 88.646 90)
-			(hide yes)
-			(show_name no)
-			(do_not_autoplace no)
-			(effects
-				(font
-					(size 1.27 1.27)
-				)
-				(justify right bottom)
-			)
-		)
-		(property "DESCRIPTION" "ON SEMICONDUCTOR - - DIODE, SCHOTTKY, 1A, 40V, DO-214AC-2"
 			(at 101.092 88.646 90)
 			(hide yes)
@@
 			)
 		)
-		(property "Value" "XIAO-ESP32-C3"
+		(property "Value" "XIAO-ESP32-S3"
 			(at 127 124.46 90)
 			(show_name no)
